File: hardware/tiny-ch32.kicad_pcb (KiCad board)
At the start: 2 copper layers, 15.2 x 27.9 mm, 17 parts, among them J1 USB_C_Receptacle_USB2.0_14P, J2 Conn_01x10, J3 Conn_01x10, U1 CH32V003FxUx, U2 XC6206PxxxMR

Commit message: Stash
Parts:
- added G*** (x2): LOGO, LOGO, F.Cu at (110.8, 120.8)
- added G*** (x2): LOGO, LOGO, F.Cu at (171.1, 102.2)
- added G***: LOGO, LOGO, F.Cu at (121.3, 96.1)
- added G***: LOGO, LOGO, F.Cu at (108.4, 97.4)
- added G*** (x2): LOGO, LOGO, B.Cu at (160.4, 96.1)
- added REF**: Icy Electronics Logo, PCM_ckl-misc:Icy Electronics Logo, B.Cu at (162.6, 106.4)
- moved C1 7.01 mm to (144.0, 97.7)
- moved C17 7.01 mm to (145.6, 90.5)
- moved J1 7.01 mm to (143.2, 83.4)
- moved J2 7.01 mm to (150.2, 84.7)
- moved J3 7.01 mm to (136.2, 107.6)
- moved R1 7.01 mm to (142.7, 96.7)
- moved R3 7.01 mm to (144.1, 89.8)
- moved C18 7.01 mm to (145.9, 95.5)
- moved D1 7.01 mm to (146.2, 98.6)
- moved D2 7.01 mm to (147.1, 93.5)
- moved JP1 7.01 mm to (145.0, 96.6)
- moved JP2 7.01 mm to (147.9, 90.8)
- moved R2 7.01 mm to (146.7, 97.1)
- moved R4 7.01 mm to (140.7, 89.8)
- moved R5 7.01 mm to (147.1, 92.6)
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Routing:
- net GND: vias 32 -> 31
